File: debugger-pcb-rev4.kicad_sch (KiCad schematic)
At the start: 37 parts, among them J1 SWD-pico, J2 SWD, J3 Conn_01x21, J6 GT-USB-7010ASV, J7 Conn_01x01, J8 Conn_01x21, Q1 MMBT2222A, Q2 MMBT5401, SW1 RESET, SW2 SSSS811101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

Commit message: more progress: final overall layout
Parts:
- removed D2: SP0503BAHT, Package_TO_SOT_SMD:SOT-143, symbol Power_Protection:SP0503BAHT
- removed TP1: VBUS, Connector_PinHeader_2.54mm:PinHeader_1x01_P2.54mm_Vertical, symbol Connector:TestPoint
- added D2, D6, D7: H7VL10B, Diode_SMD:D_SOD-882, symbol Device:D_TVS
- added J4: Conn_01x02, Connector_PinHeader_2.54mm:PinHeader_1x02_P2.54mm_Horizontal, symbol Connector_Generic:Conn_01x02
- F1: value SMD1210-050-16V -> BSMD0805-050-24V; footprint Fuse:Fuse_1210_3225Metric -> Fuse:Fuse_0805_2012Metric; JLC P/N C70095 -> (none)
- J1: symbol Connector_Generic:Conn_01x03 -> Connector_Generic_MountingPin:Conn_01x03_MountingPin
Connections:
- net GND: now also D2.1 (A1), D6.1 (A1), D7.1 (A1)
- net USB_DM: now also D6.2 (A2)
- net USB_DP: now also D2.2 (A2)
- net at F1.2, J6.A4 (VBUS), J6.A9 (VBUS)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: now also D7.2 (A2)
- net USART2_RX renamed ACIA_RX
- net ACIA_RX: now also J4.2 (Pin_2)
- net USART2_TX renamed ACIA_TX
- net ACIA_TX: now also J4.1 (Pin_1)
- no-connect marks 8 -> 9
Other:
- moved on the sheet: J2

Commit message: close to final
Parts:
- added J5, J9: Conn_01x02, Connector_PinHeader_2.54mm:PinHeader_1x02_P2.54mm_Vertical, symbol Connector_Generic:Conn_01x02
- F1: value BSMD0805-050-24V -> 0402L050SL; footprint Fuse:Fuse_0805_2012Metric -> Fuse:Fuse_0402_1005Metric
- J1: footprint Connector_JST:JST_SH_SM03B-SRSS-TB_1x03-1MP_P1.00mm_Horizontal -> custom:JST_SH_BM03B-SRSS-TB_1x03-1MP_P1.00mm_Vertical
- J2: now not fitted
- J4: footprint Connector_PinHeader_2.54mm:PinHeader_1x02_P2.54mm_Horizontal -> Connector_PinHeader_2.54mm:PinHeader_1x02_P2.54mm_Vertical
- Q1, Q2: footprint Package_TO_SOT_SMD:SOT-523 -> custom:SOT-523
- SW1: value RESET -> RST
Connections:
- net USART1_RX is gone; now on net ACIA_RX: U1.43 (PA10)
- net USART1_TX is gone; now on net ACIA_TX: U1.42 (PA9)
- net ACIA_RX: now also J4.1 (Pin_1); no longer J4.2 (Pin_2), U1.17 (PA3)
- net ACIA_TX: now also J4.2 (Pin_2); no longer J4.1 (Pin_1), U1.16 (PA2)
- net SWCLK: now also J1.1 (Pin_1); no longer J1.3 (Pin_3)
- net SWDIO: now also J1.3 (Pin_3); no longer J1.1 (Pin_1)
- net PB1: now reaches U1.27 (PB1)
- net PB1: now also J9.1 (Pin_1)
- net PB12: now reaches U1.33 (PB12)
- net PB12: now also J9.2 (Pin_2)
- new net PA2: J5.1 (Pin_1), U1.16 (PA2)
- new net PA3: J5.2 (Pin_2), U1.17 (PA3)

Commit message: design reviewed and part #s added
Parts:
- C1, C2, C3, C6, C7: JLC P/N (none) -> C1525
- C4: JLC P/N C15850 -> C15525
- C5: JLC P/N C49678 -> C1525
- D1: value R6GHBHC -> R6GHBHC-A01/2T; JLC P/N (none) -> C60105
- D2, D6, D7: JLC P/N (none) -> C20615787
- F1: JLC P/N (none) -> C206938
- J1: JLC P/N (none) -> C3029333
- Q1: JLC P/N C8512 -> C22468359
- Q2: symbol Device:Q_PNP_BEC -> Transistor_BJT:Q_PNP_BEC; JLC P/N C8326 -> C42415188
- R1: JLC P/N (none) -> C25744
- R10, R5: value 470 -> 330; JLC P/N (none) -> C25104
- R2, R4: JLC P/N C27834 -> C25905
- R3: value 470 -> 220; JLC P/N (none) -> C25091
- R6, R8: JLC P/N C17414 -> C25744
- R7, R9: JLC P/N C17513 -> C11702
- SW1, SW3, SW4: JLC P/N C318884 -> C720477
- U1: JLC P/N (none) -> C2683478
Connections:
- net GND: now also J6.S1 (SHIELD)
- no-connect marks 9 -> 8
Other:
- note added: "TODO: VALUES"
Changed lines of the file:
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@@
 		)
 	)
+	(text "TODO: VALUES"
+		(exclude_from_sim no)
+		(at 134.62 119.38 0)
+		(effects
+			(font
+				(size 1.27 1.27)
+			)
+		)
+	)
 	(text "PHI1O"
 		(exclude_from_sim no)
@@
 	)
 	(no_connect
-		(at 114.3 191.77)
-	)
-	(no_connect
 		(at 245.11 105.41)
 	)
@@
 	(wire
 		(pts
+			(xy 114.3 191.77) (xy 121.92 191.77)
+		)
+		(stroke
+			(width 0)
+			(type default)
+		)
+	)
+	(wire
+		(pts
 			(xy 125.73 191.77) (xy 147.32 191.77)
 		)
@@
 			)
 		)
+		(property "JLC P/N" "C20615787"
+			(at 147.32 186.69 0)
+			(effects
+				(font
+					(size 1.27 1.27)
+				)
+			)
+		)
 		(pin "2"
 		)
@@
 			)
 		)
-		(property "JLC P/N" "C27834"
+		(property "JLC P/N" "C25905"
 			(at 140.97 158.75 0)
 			(effects
@@
 			)
 		)
+		(property "JLC P/N" "C1525"
+			(at 64.77 25.4 0)
+			(effects
+				(font
+					(size 1.27 1.27)
+				)
+			)
+		)
 		(pin "1"
 		)
@@
 			)
 		)
+		(property "JLC P/N" "C2683478"
+			(at 72.39 99.06 0)
+			(effects
+				(font
+					(size 1.27 1.27)
+				)
+				(hide yes)
+			)
+		)
 		(pin "29"
 		)
@@
 			)
 		)
-		(property "Value" "R6GHBHC"
+		(property "Value" "R6GHBHC-A01/2T"
 			(at 142.24 95.25 0)
 			(effects
@@
 			)
 		)
+		(property "JLC P/N" "C60105"
+			(at 142.24 106.68 0)
+			(effects
+				(font
+					(size 1.27 1.27)
+				)
+				(hide yes)
+			)
+		)
 		(pin "2"
 		)
@@
 			)
 		)
+		(property "JLC P/N" "C1525"
+			(at 53.34 25.4 0)
+			(effects
+				(font
+					(size 1.27 1.27)
+				)
+			)
+		)
 		(pin "1"
 		)
@@
 			)
 		)
-		(property "JLC P/N" ""
+		(property "JLC P/N" "C206938"
 			(at 158.75 147.32 0)
 			(effects
@@
 			)
 		)
-		(property "JLC P/N" "C318884"
+		(property "JLC P/N" "C720477"
 			(at 107.95 129.54 0)
 			(effects
@@
 			)
 		)
-		(property "JLC P/N" "C17414"
+		(property "JLC P/N" "C25744"
 			(at 248.92 45.72 0)
 			(effects
@@
 			)
 		)
-		(property "Value" "470"
+		(property "Value" "220"
 			(at 137.16 104.14 90)
 			(effects
@@
 			)
 		)
+		(property "JLC P/N" "C25091"
+			(at 133.35 106.68 90)
+			(effects
+				(font
+					(size 1.27 1.27)
+				)
+				(hide yes)
+			)
+		)
 		(pin "1"
 		)
@@
 			)
 		)
+		(property "JLC P/N" "C25744"
+			(at 35.56 67.31 0)
+			(effects
+				(font
+					(size 1.27 1.27)
+				)
+			)
+		)
 		(pin "1"
 		)
@@
 			)
 		)
-		(property "JLC P/N" "C27834"
+		(property "JLC P/N" "C25905"
 			(at 140.97 161.29 0)
 			(effects
@@
 			)
 		)
-		(property "JLC P/N" "C8512"
+		(property "JLC P/N" "C22468359"
 			(at 232.41 45.72 0)
 			(effects
@@
 			)
 		)
+		(property "JLC P/N" "C1525"
+			(at 41.91 25.4 0)
+			(effects
+				(font
+					(size 1.27 1.27)
+				)
+			)
+		)
 		(pin "1"
 		)
@@
 			)
 		)
-		(property "JLC P/N" "C318884"
+		(property "JLC P/N" "C720477"
 			(at 49.53 49.53 0)
 			(effects
@@
 			)
 		)
-		(property "Value" "470"
+		(property "Value" "330"
 			(at 137.16 109.22 90)
 			(effects
@@
 			)
 		)
+		(property "JLC P/N" "C25104"
+			(at 133.35 111.76 90)
+			(effects
+				(font
+					(size 1.27 1.27)
+				)
+				(hide yes)
+			)
+		)
 		(pin "1"
 		)
@@
 			)
 		)
-		(property "JLC P/N" "C17513"
+		(property "JLC P/N" "C11702"
 			(at 229.87 36.83 0)
 			(effects
@@
 			)
 		)
+		(property "JLC P/N" "C1525"
+			(at 19.05 25.4 0)
+			(effects
+				(font
+					(size 1.27 1.27)
+				)
+			)
+		)
 		(pin "1"
 		)
@@
 			)
 		)
+		(property "Sim.Pins" "1=K 2=A"
+			(at 260.35 36.83 0)
+			(effects
+				(font
+					(size 1.27 1.27)
+				)
+				(hide yes)
+			)
+		)
 		(pin "2"
 		)
@@
 			)
 		)
+		(property "JLC P/N" "C20615787"
+			(at 165.1 186.69 0)
+			(effects
+				(font
+					(size 1.27 1.27)
+				)
+			)
+		)
 		(pin "2"
 		)
@@
 			)
 		)
-		(property "JLC P/N" "C15850"
+		(property "JLC P/N" "C15525"
 			(at 165.1 153.67 0)
 			(effects
@@
 			)
 		)
-		(property "Value" "470"
+		(property "Value" "330"
 			(at 137.16 99.06 90)
 			(effects
@@
 			)
 		)
+		(property "JLC P/N" "C25104"
+			(at 133.35 101.6 90)
+			(effects
+				(font
+					(size 1.27 1.27)
+				)
+				(hide yes)
+			)
+		)
 		(pin "1"
 		)
@@
 			)
 		)
-		(property "JLC P/N" "C49678"
+		(property "JLC P/N" "C1525"
 			(at 175.26 153.67 0)
 			(effects
@@
 			)
 		)
-		(property "JLC P/N" "C17513"
+		(property "JLC P/N" "C11702"
 			(at 260.35 54.61 0)
 			(effects
@@
 			)
 		)
-		(property "JLC P/N" "C318884"
+		(property "JLC P/N" "C720477"
 			(at 107.95 127 0)
 			(effects
@@
 			)
 		)
+		(property "JLC P/N" "C3029333"
+			(at 119.38 31.75 0)
+			(effects
+				(font
+					(size 1.27 1.27)
+				)
+			)
+		)
 		(pin "3"
 		)
@@
 	)
 	(symbol
+		(lib_name "LED_1")
 		(lib_id "Device:LED")
 		(at 229.87 54.61 270)
@@
 			)
 		)
+		(property "Sim.Pins" "1=K 2=A"
+			(at 229.87 54.61 0)
+			(effects
+				(font
+					(size 1.27 1.27)
+				)
+				(hide yes)
+			)
+		)
 		(pin "1"
 		)
@@
 			)
 		)
+		(property "JLC P/N" "C20615787"
+			(at 156.21 186.69 0)
+			(effects
+				(font
+					(size 1.27 1.27)
+				)
+			)
+		)
 		(pin "2"
 		)
@@
 	)
 	(symbol
-		(lib_id "Device:Q_PNP_BEC")
+		(lib_id "Transistor_BJT:Q_PNP_BEC")
 		(at 257.81 45.72 0)
 		(mirror x)
@@
 			)
 		)
-		(property "JLC P/N" "C8326"
+		(property "JLC P/N" "C42415188"
 			(at 257.81 45.72 0)
 			(effects
@@
 			)
 		)
+		(property "JLC P/N" "C1525"
+			(at 30.48 25.4 0)
+			(effects
+				(font
+					(size 1.27 1.27)
+				)
+			)
+		)
 		(pin "1"
 		)
@@
 			)
 		)
-		(property "JLC P/N" "C17414"
+		(property "JLC P/N" "C25744"
 			(at 241.3 45.72 0)
 			(effects

Commit message: jlc bom script, fix components
Parts:
- J2, J3, J4, J5, J7, J8, J9, JP1: now left out of the parts list
- Q1: JLC P/N C22468359 -> C94417
- Q2: JLC P/N C42415188 -> C2836079
Changed lines of the file:
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@@
 			)
 		)
-		(property "Description" "Resistor, US symbol"
+		(property "Description" "Resistor"
 			(at 140.97 158.75 0)
 			(effects
@@
 			)
 		)
-		(property "Description" ""
+		(property "Description" "32-bit ARM microcontroller"
 			(at 72.39 99.06 0)
 			(effects
@@
 		(unit 1)
 		(exclude_from_sim yes)
-		(in_bom yes)
+		(in_bom no)
 		(on_board yes)
 		(dnp no)
@@
 			)
 		)
-		(property "Description" "Resistor, US symbol"
+		(property "Description" "Resistor"
 			(at 248.92 45.72 0)
 			(effects
@@
 		(unit 1)
 		(exclude_from_sim no)
-		(in_bom yes)
+		(in_bom no)
 		(on_board yes)
 		(dnp no)
@@
 			)
 		)
-		(property "Description" "Resistor, US symbol"
+		(property "Description" "Resistor"
 			(at 140.97 161.29 0)
 			(effects
@@
 			)
 		)
-		(property "JLC P/N" "C22468359"
+		(property "JLC P/N" "C94417"
 			(at 232.41 45.72 0)
 			(effects
@@
 		(unit 1)
 		(exclude_from_sim no)
-		(in_bom yes)
+		(in_bom no)
 		(on_board yes)
 		(dnp no)
@@
 		(unit 1)
 		(exclude_from_sim no)
-		(in_bom yes)
+		(in_bom no)
 		(on_board yes)
 		(dnp yes)
@@
 			)
 		)
-		(property "Description" "Resistor, US symbol"
+		(property "Description" "Resistor"
 			(at 229.87 36.83 0)
 			(effects
@@
 		(unit 1)
 		(exclude_from_sim no)
-		(in_bom yes)
+		(in_bom no)
 		(on_board yes)
 		(dnp no)
@@
 			)
 		)
-		(property "Description" "Resistor, US symbol"
+		(property "Description" "Resistor"
 			(at 260.35 54.61 0)
 			(effects
@@
 		(unit 1)
 		(exclude_from_sim no)
-		(in_bom yes)
+		(in_bom no)
 		(on_board yes)
 		(dnp yes)
@@
 			)
 		)
-		(property "JLC P/N" "C42415188"
+		(property "JLC P/N" "C2836079"
 			(at 257.81 45.72 0)
 			(effects
@@
 		(unit 1)
 		(exclude_from_sim no)
-		(in_bom yes)
+		(in_bom no)
 		(on_board yes)
 		(dnp yes)
@@
 		(unit 1)
 		(exclude_from_sim no)
-		(in_bom yes)
+		(in_bom no)
 		(on_board yes)
 		(dnp no)
@@
 			)
 		)
-		(property "Description" "Resistor, US symbol"
+		(property "Description" "Resistor"
 			(at 241.3 45.72 0)
 			(effects

Commit message: as ordered for batch 1
Parts:
- J3, J8: footprint Connector_PinHeader_2.54mm:PinHeader_1x21_P2.54mm_Vertical -> custom:PinHeader_1x21_P2.54mm_Vertical_nosilk
Changed lines of the file:
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@@
 			)
 		)
-		(property "Description" "32-bit ARM microcontroller"
+		(property "Description" ""
 			(at 72.39 99.06 0)
 			(effects
@@
 			)
 		)
-		(property "Footprint" "Connector_PinHeader_2.54mm:PinHeader_1x21_P2.54mm_Vertical"
+		(property "Footprint" "custom:PinHeader_1x21_P2.54mm_Vertical_nosilk"
 			(at 231.14 125.73 0)
 			(effects
@@
 			)
 		)
-		(property "Footprint" "Connector_PinHeader_2.54mm:PinHeader_1x21_P2.54mm_Vertical"
+		(property "Footprint" "custom:PinHeader_1x21_P2.54mm_Vertical_nosilk"
 			(at 240.03 125.73 0)
 			(effects
