File: pcb/debugger-pcb-rev4.kicad_pcb (KiCad board)
At the start: 4 copper layers, 17.8 x 68.6 mm, 42 parts, among them J1 SWD-pico, J2 SWD, J3 Conn_01x21, J4 Conn_01x02, J5 Conn_01x02, J6 GT-USB-7010ASV, J7 Conn_01x01, J8 Conn_01x21, J9 Conn_01x02, Q1 MMBT2222A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

Commit message: 4.1 board revisions done?
Parts:
- removed J2: SWD, Connector_PinHeader_2.54mm:PinHeader_1x03_P2.54mm_Vertical
- removed J5: Conn_01x02, Connector_PinHeader_2.54mm:PinHeader_1x02_P2.54mm_Vertical
- removed JP1: BOOT0, Jumper:SolderJumper-2_P1.3mm_Open_RoundedPad1.0x1.5mm
- added C8: 10pF, Capacitor_SMD:C_0402_1005Metric, F.Cu at (198.8, 63.2)
- added C9: 10pF, Capacitor_SMD:C_0402_1005Metric, F.Cu at (196.6, 64.2)
- added SW5: BOOT0, custom:SW_Push_SPST_TS-1088, F.Cu at (198.8, 60.9)
- added TP1: DM, TestPoint:TestPoint_Pad_1.0x1.0mm, F.Cu at (197.8, 83.2)
- added TP2: DP, TestPoint:TestPoint_Pad_1.0x1.0mm, F.Cu at (197.8, 85.2)
- added Y1: 16MHz, Crystal:Crystal_SMD_3225-4Pin_3.2x2.5mm, F.Cu at (199.3, 65.4)
- moved J1 6.86 mm to (196.8, 54.4), turned to 0 degrees
- moved R1 2.02 mm to (200.8, 63.2)
Connections:
- U1 pad 16: /PA2 -> /RESB
- U1 pad 17: /PA3 -> /EEPROM_~{PROG}
- U1 pad 5: /RESB -> Net-(U1-PD0)
- U1 pad 6: /EEPROM_~{PROG} -> Net-(U1-PD1)
Routing:
- net /PA2: track 24.3 -> 0.00 mm, vias 1 -> 0
- net /PA3: track 20.4 -> 0.00 mm, vias 2 -> 0
- net Net-(U1-PD0): track 0.00 -> 7.46 mm
- net /RESB: track 30.0 -> 37.0 mm, vias 0 -> 1
- net /EEPROM_~{PROG}: track 32.5 -> 39.0 mm, vias 0 -> 2
- net Net-(U1-PD1): track 0.00 -> 5.36 mm
- net /SWCLK: track 32.9 -> 28.0 mm, vias 1 -> 2
- net Net-(U1-BOOT0): track 11.5 -> 15.5 mm
- net /A15: track 19.9 -> 17.0 mm
- net /SWDIO: track 25.4 -> 27.0 mm, vias 1 -> 2
- net /USB_DP: track 32.2 -> 33.0 mm
- net GND: track 54.7 -> 55.1 mm, vias 16 -> 47
- net +5V: track 29.1 -> 29.0 mm, vias 9 -> 10
Other:
- board text added: "6502 Debugger"
- board text added: "H"
- board text added: "L"
- board text added: "rev4.1"
- board text removed: "A3"
- board text removed: "rev4.0"
