File: pcb/debugger-pcb-rev4.kicad_sch (KiCad schematic)
At the start: 41 parts, among them J1 SWD-pico, J2 SWD, J3 Conn_01x21, J4 Conn_01x02, J5 Conn_01x02, J6 GT-USB-7010ASV, J7 Conn_01x01, J8 Conn_01x21, J9 Conn_01x02, Q1 MMBT2222A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

Commit message: 4.1 board revisions done?
Parts:
- removed J2: SWD, Connector_PinHeader_2.54mm:PinHeader_1x03_P2.54mm_Vertical, symbol Connector_Generic:Conn_01x03
- removed J5: Conn_01x02, Connector_PinHeader_2.54mm:PinHeader_1x02_P2.54mm_Vertical, symbol Connector_Generic:Conn_01x02
- removed JP1: BOOT0, Jumper:SolderJumper-2_P1.3mm_Open_RoundedPad1.0x1.5mm, symbol Jumper:Jumper_2_Small_Open
- added C8, C9: 10pF, Capacitor_SMD:C_0402_1005Metric, symbol Device:C
- added SW5: BOOT0, custom:SW_Push_SPST_TS-1088, symbol Switch:SW_Push
- added TP1: DM, TestPoint:TestPoint_Pad_1.0x1.0mm, symbol Connector:TestPoint
- added TP2: DP, TestPoint:TestPoint_Pad_1.0x1.0mm, symbol Connector:TestPoint
- added Y1: 16MHz, Crystal:Crystal_SMD_3225-4Pin_3.2x2.5mm, symbol Device:Crystal_GND24
- D4: JLC P/N C965817 -> C98225
Connections:
- net PA2 is gone; now on net RESB: U1.16 (PA2)
- net PA3 is gone; now on net EEPROM_~{PROG}: U1.17 (PA3)
- net +5V: now also SW5.1
- net EEPROM_~{PROG}: no longer U1.6 (PD1)
- net GND: now also C8.1, C9.1, Y1.2, Y1.4
- net RESB: no longer U1.5 (PD0)
- net USB_DM: now also TP1.1
- net USB_DP: now also TP2.1
- net at R1.1, U1.60 (BOOT0): now also SW5.2
- new net: C8.2, U1.5 (PD0), Y1.3
- new net: C9.2, U1.6 (PD1), Y1.1
Other:
- note added: "NC"
- note removed: "TODO: VALUES"
- moved on the sheet: R1
